File: ambush.brd (EAGLE design)
At the start: 100 x 100 mm, 96 parts, among them IC1 LM555N, IC10 LM555N, IC11 7430N, IC12 7400N, IC13 LM386N-3, IC14 74LS93N, IC15 74LS93N, IC16 7410N, IC17 7402N, IC18 7402N, IC19 7486N, IC2 7404N, IC20 74125N, IC21 7400N, IC22 LM555N, IC23 LM555N, IC24 7400N, IC25 LM555N, IC26 LM555N, IC3 LM555N, IC4 LM555N, IC5 7404N, IC6 74LS93N, IC7 LM555N, IC8 LM555N, IC9 74LS93N, T1 2N3904, T2 2N3904, T3 2N3904, T4 2N3904, T5 2N3904, T6 2N3904, Y1 14.3 MHz

Commit message: -finished control board
Parts:
- added C24, C27, C28, C30: 10nF, resistor:C025-040X050
- added C25, C26, C31, C32, C34, C35: 100nF, resistor:C025-040X050
- added C29: 47nF, resistor:C025-040X050
- added C33: 200nF, resistor:C025-040X050
- added IC27: 74S20N, 74xx-us:DIL14
- added IC28, IC37: 7404N, 74xx-us:DIL14
- added IC29, IC34, IC35: LM555N, linear:DIL08
- added IC30: 7400N, 74xx-us:DIL14
- added IC31: 7475N, 74xx-us:DIL16
- added IC32, IC33: 7485N, 74xx-us:DIL16
- added IC36: 7402N, 74xx-us:DIL14
- added MOV_POT: 500k, pot:3RP/1610N
- added R36: 470k, resistor:0207/10
- added R37, R42, R43: 1M, resistor:0207/10
- added R38, R39, R41, R44, R45: 470, resistor:0207/10
- added R40: 3.3k, resistor:0207/10
Connections:
- new net !128H: IC27.2
- new net !256H: IC27.1
- new net !32H: IC27.5
- new net !64H: IC27.4
- new net !GH: IC24.12, IC28.2
- new net !GV: IC28.4, IC28.5, IC30.1
- new net BG_FLASH: IC26.3, IC36.5
- new net LOAD\: IC24.8
- new net N$67: C24.1, IC26.5
- new net N$68: C25.1, IC26.2, IC26.6, R36.2
- new net N$69: IC26.7, R36.1, R37.2
- new net N$70: C26.1, IC24.6
- new net N$71: C26.2, IC2.13, R38.1
- new net N$72: C27.2, IC24.11
- new net N$73: IC2.12, IC24.5, IC24.9
- new net N$74: C27.1, IC28.1, R39.1
- new net N$75: IC29.3, IC30.2
- new net N$76: C28.1, IC29.5
- new net N$77: C30.2, IC30.3
- new net N$78: C29.1, IC29.6, IC29.7, R40.2
- new net N$79: C29.2
- new net N$80: MOV_POT.1, R40.1
- new net N$81: C30.1, IC28.3, R41.1
- new net N$82: IC31.1, IC32.10
- new net N$83: IC31.15, IC33.10
- new net N$84: IC31.10, IC32.13, IC33.12
- new net N$85: IC28.6, IC30.5
- new net N$86: IC30.12, IC30.4, IC32.6
- new net N$87: IC28.9, IC30.6, IC34.2
- new net N$88: IC31.9, IC32.15, IC33.13
- new net N$89: C31.2, IC34.5
- new net N$90: C32.2, IC35.5
- new net N$91: C33.2, IC34.6, IC34.7, R42.1
- new net N$92: C34.2, IC35.6, IC35.7, R43.1
- new net N$93: C35.2, IC34.3, R44.2
- new net N$94: C35.1, IC35.2, R45.2
- new net N$95: IC30.13, IC33.6
- new net N$96: IC30.10, IC35.3
- new net N$97: IC30.11, IC36.6
- new net START_PULSE: IC2.8, IC21.9, IC22.2, IC24.10
- net !GHIT: now also IC30.8
- net +5V: now also IC29.8, IC34.4, IC34.8, IC35.4, IC35.8, MOV_POT.3, R37.1, R42.2, R43.2, R44.1, R45.1
- net 128H: now also IC33.1
- net 128V: now also IC32.1
- net 16H: now also IC33.9
- net 16V: now also IC32.9
- net 1V: now also IC31.2
- net 2V: now also IC31.3
- net 32H: now also IC33.11
- net 32V: now also IC32.11
- net 4V: now also IC31.6
- net 64H: now also IC33.14
- net 64V: now also IC32.14
- net 8V: now also IC31.7
- net GND: now also C24.2, C25.2, C28.2, C31.1, C32.1, C33.1, C34.1, IC27.7, IC28.7, IC29.1, IC30.7, IC31.12, IC32.2, IC32.4, IC32.8, IC33.15, IC33.2, IC33.4, IC33.8, IC34.1, IC35.1, IC36.7, IC37.7, R38.2, R39.2, R41.2
- net GV=BV: now also IC28.8, IC30.9
- net LOAD: now also IC31.13, IC31.4
- net N$52: now also IC24.13, IC27.6; no longer IC2.8, IC21.9, IC22.2
- net N$66: now also IC24.4
- net VCC: now also IC27.14, IC28.14, IC30.14, IC31.5, IC32.16, IC33.16, IC36.14, IC37.14
- net VRST: now also IC29.2, IC29.4

Commit message: -finished copying my modified schematics from paper to eagle
Connections:
- new net N$100: IC28.11, IC36.10
- new net N$98: IC36.4, IC36.8
- new net N$99: IC36.1, IC36.9
- net !128H: now also IC37.2
- net !256H: now also IC28.12
- net !32H: now also IC37.6
- net !64H: now also IC37.4
- net !GH: now also IC36.2
- net !GV: now also IC36.3
- net 128H: now also IC37.1
- net 256H: now also IC28.13
- net 32H: now also IC37.5
- net 64H: now also IC37.3
- net GAME_VID: now also IC28.10
Changed lines of the file:
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@@
 <contactref element="IC12" pad="12"/>
 <contactref element="IC33" pad="11"/>
+<contactref element="IC37" pad="5"/>
 <wire x1="20.08" y1="-889.19" x2="12.46" y2="-1011.19" width="0" layer="19" extent="1-1"/>
 <wire x1="3.81" y1="3.81" x2="12.46" y2="-1011.19" width="0" layer="19" extent="1-1"/>
+<wire x1="2.54" y1="-3.81" x2="3.81" y2="3.81" width="0" layer="19" extent="1-1"/>
 </signal>
 <signal name="64H">
@@
 <contactref element="IC12" pad="1"/>
 <contactref element="IC33" pad="14"/>
+<contactref element="IC37" pad="3"/>
 <wire x1="20.08" y1="-946.81" x2="7.38" y2="-1018.81" width="0" layer="19" extent="1-1"/>
 <wire x1="22.62" y1="-889.19" x2="20.08" y2="-946.81" width="0" layer="19" extent="1-1"/>
-<wire x1="-3.81" y1="3.81" x2="7.38" y2="-1018.81" width="0" layer="19" extent="1-1"/>
+<wire x1="-2.54" y1="-3.81" x2="7.38" y2="-1018.81" width="0" layer="19" extent="1-1"/>
+<wire x1="-3.81" y1="3.81" x2="-2.54" y2="-3.81" width="0" layer="19" extent="1-1"/>
 </signal>
 <signal name="128H">
@@
 <contactref element="IC11" pad="5"/>
 <contactref element="IC33" pad="1"/>
+<contactref element="IC37" pad="1"/>
 <wire x1="15" y1="-889.19" x2="17.54" y2="-946.81" width="0" layer="19" extent="1-1"/>
 <wire x1="14.73" y1="-847.19" x2="15" y2="-889.19" width="0" layer="19" extent="1-1"/>
 <wire x1="-8.89" y1="-3.81" x2="17.54" y2="-946.81" width="0" layer="19" extent="1-1"/>
+<wire x1="-7.62" y1="-3.81" x2="-8.89" y2="-3.81" width="0" layer="19" extent="1-1"/>
 </signal>
 <signal name="HRST">
@@
 <contactref element="V1" pad="9"/>
 <contactref element="IC11" pad="4"/>
+<contactref element="IC28" pad="13"/>
 <wire x1="24.89" y1="-847.19" x2="15" y2="-946.81" width="0" layer="19" extent="1-1"/>
+<wire x1="5.92" y1="-1809.19" x2="15" y2="-946.81" width="0" layer="19" extent="1-1"/>
 </signal>
 <signal name="N$26">
@@
 <contactref element="IC18" pad="3"/>
 <contactref element="IC18" pad="2"/>
+<contactref element="IC28" pad="10"/>
 <wire x1="12.46" y1="-1176.81" x2="9.92" y2="-1176.81" width="0" layer="19" extent="1-1"/>
+<wire x1="13.54" y1="-1809.19" x2="9.92" y2="-1176.81" width="0" layer="19" extent="1-1"/>
 </signal>
 <signal name="N$42">
@@
 <signal name="!256H">
 <contactref element="IC27" pad="1"/>
+<contactref element="IC28" pad="12"/>
+<wire x1="3.38" y1="-1795.81" x2="8.46" y2="-1809.19" width="0" layer="19" extent="1-1"/>
 </signal>
 <signal name="!128H">
 <contactref element="IC27" pad="2"/>
+<contactref element="IC37" pad="2"/>
+<wire x1="-5.08" y1="-3.81" x2="5.92" y2="-1795.81" width="0" layer="19" extent="1-1"/>
 </signal>
 <signal name="!64H">
 <contactref element="IC27" pad="4"/>
+<contactref element="IC37" pad="4"/>
+<wire x1="0" y1="-3.81" x2="11" y2="-1795.81" width="0" layer="19" extent="1-1"/>
 </signal>
 <signal name="!32H">
 <contactref element="IC27" pad="5"/>
+<contactref element="IC37" pad="6"/>
+<wire x1="5.08" y1="-3.81" x2="13.54" y2="-1795.81" width="0" layer="19" extent="1-1"/>
 </signal>
 <signal name="N$72">
@@
 <contactref element="IC24" pad="12"/>
 <contactref element="IC28" pad="2"/>
+<contactref element="IC36" pad="2"/>
 <wire x1="5.92" y1="-1816.81" x2="8.46" y2="-1525.19" width="0" layer="19" extent="1-1"/>
+<wire x1="-5.08" y1="-3.81" x2="8.46" y2="-1525.19" width="0" layer="19" extent="1-1"/>
 </signal>
 <signal name="N$76">
@@
 <contactref element="IC28" pad="4"/>
 <contactref element="IC28" pad="5"/>
+<contactref element="IC36" pad="3"/>
 <wire x1="11" y1="-1816.81" x2="3.38" y2="-1955.81" width="0" layer="19" extent="1-1"/>
 <wire x1="13.54" y1="-1816.81" x2="11" y2="-1816.81" width="0" layer="19" extent="1-1"/>
+<wire x1="-2.54" y1="-3.81" x2="3.38" y2="-1955.81" width="0" layer="19" extent="1-1"/>
 </signal>
 <signal name="N$82">
@@
 <wire x1="5.08" y1="-3.81" x2="11" y2="-1948.19" width="0" layer="19" extent="1-1"/>
 </signal>
+<signal name="N$98">
+<contactref element="IC36" pad="4"/>
+<contactref element="IC36" pad="8"/>
+<wire x1="0" y1="-3.81" x2="7.62" y2="3.81" width="0" layer="19" extent="1-1"/>
+</signal>
+<signal name="N$99">
+<contactref element="IC36" pad="1"/>
+<contactref element="IC36" pad="9"/>
+<wire x1="5.08" y1="3.81" x2="-7.62" y2="-3.81" width="0" layer="19" extent="1-1"/>
+</signal>
+<signal name="N$100">
+<contactref element="IC36" pad="10"/>
+<contactref element="IC28" pad="11"/>
+<wire x1="2.54" y1="3.81" x2="11" y2="-1809.19" width="0" layer="19" extent="1-1"/>
+</signal>
 </signals>

Commit message: -added a feature so the paddle disappears when the game isn't started -made it so the player can't be killed by the bad guy while the bad guy is flashing
Parts:
- added IC38: 7400N, 74xx-us:DIL14
Connections:
- removed net N$55: IC21.13, IC22.3
- removed net N$79: C29.2
- new net !GDEAD: IC10.2, IC22.4, IC37.8, R20.1
- new net BDEAD: IC24.4, IC25.3, IC26.4, IC38.1
- new net GAMEACTIVE: IC21.13, IC22.3, IC38.4
- new net N$101: IC37.11, IC38.6
- new net N$102: IC29.2, IC29.4, IC37.10
- net !GHIT: now also IC38.2; no longer IC10.2, IC22.4, R20.1
- net GND: now also C29.2, IC38.7
- net N$66: now also IC37.9, IC38.3; no longer IC24.4, IC25.3, IC26.4
- net VCC: now also IC38.14
- net VRST: now also IC38.5; no longer IC29.2, IC29.4
Changed lines of the file:
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@@
 <element name="IC36" library="74xx-us" library_urn="urn:adsk.eagle:library:88" package="DIL14" package3d_urn="urn:adsk.eagle:package:2921/1" value="7402N" x="0" y="0"/>
 <element name="IC37" library="74xx-us" library_urn="urn:adsk.eagle:library:88" package="DIL14" package3d_urn="urn:adsk.eagle:package:2921/1" value="7404N" x="0" y="0"/>
+<element name="IC38" library="74xx-us" library_urn="urn:adsk.eagle:library:88" package="DIL14" package3d_urn="urn:adsk.eagle:package:2921/1" value="7400N" x="0" y="0"/>
 </elements>
 <signals>
@@
 <contactref element="IC36" pad="7"/>
 <contactref element="IC37" pad="7"/>
+<contactref element="IC38" pad="7"/>
+<contactref element="C29" pad="2"/>
 <wire x1="6.27" y1="-1511" x2="18.62" y2="-1532.81" width="0" layer="19" extent="1-1"/>
 <wire x1="3.19" y1="-1553.81" x2="18.62" y2="-1532.81" width="0" layer="19" extent="1-1"/>
@@
 <wire x1="3.19" y1="-1866.81" x2="13.08" y2="-1845" width="0" layer="19" extent="1-1"/>
 <wire x1="6.27" y1="-1881" x2="3.19" y2="-1866.81" width="0" layer="19" extent="1-1"/>
+<wire x1="6.27" y1="-1895" x2="6.27" y2="-1881" width="0" layer="19" extent="1-1"/>
 <wire x1="22.62" y1="-1098.81" x2="22.62" y2="-1155.81" width="0" layer="19" extent="1-1"/>
 <wire x1="14.81" y1="-1039.81" x2="22.62" y2="-1098.81" width="0" layer="19" extent="1-1"/>
 <wire x1="9.73" y1="-1039.81" x2="14.81" y2="-1039.81" width="0" layer="19" extent="1-1"/>
 <wire x1="22.62" y1="-1018.81" x2="14.81" y2="-1039.81" width="0" layer="19" extent="1-1"/>
+<wire x1="18.62" y1="-1955.81" x2="6.27" y2="-1895" width="0" layer="19" extent="1-1"/>
+<wire x1="13.08" y1="-1984" x2="18.62" y2="-1955.81" width="0" layer="19" extent="1-1"/>
+<wire x1="-8.27" y1="-1998" x2="13.08" y2="-1984" width="0" layer="19" extent="1-1"/>
 <wire x1="22.62" y1="-946.81" x2="22.62" y2="-1018.81" width="0" layer="19" extent="1-1"/>
 <wire x1="17.54" y1="-889.19" x2="22.62" y2="-946.81" width="0" layer="19" extent="1-1"/>
@@
 <wire x1="29.21" y1="-593.09" x2="7.62" y2="-593.09" width="0" layer="19" extent="1-1"/>
 <wire x1="31.75" y1="-571.5" x2="29.21" y2="-593.09" width="0" layer="19" extent="1-1"/>
-<wire x1="18.62" y1="-1955.81" x2="6.27" y2="-1881" width="0" layer="19" extent="1-1"/>
-<wire x1="13.08" y1="-1984" x2="18.62" y2="-1955.81" width="0" layer="19" extent="1-1"/>
-<wire x1="-8.27" y1="-1998" x2="13.08" y2="-1984" width="0" layer="19" extent="1-1"/>
 <wire x1="11.9888" y1="-447.04" x2="31.75" y2="-571.5" width="0" layer="19" extent="1-1"/>
 <wire x1="7.62" y1="-237.49" x2="11.9888" y2="-447.04" width="0" layer="19" extent="1-1"/>
@@
 </signal>
 <signal name="!GHIT">
-<contactref element="IC10" pad="2"/>
-<contactref element="R20" pad="1"/>
-<contactref element="IC22" pad="4"/>
+<contactref element="IC38" pad="2"/>
 <contactref element="IC30" pad="8"/>
-<wire x1="31.75" y1="-673.1" x2="31.75" y2="-717.55" width="0" layer="19" extent="1-1"/>
-<wire x1="10.81" y1="-1332.81" x2="31.75" y2="-717.55" width="0" layer="19" extent="1-1"/>
-<wire x1="18.62" y1="-1948.19" x2="10.81" y2="-1332.81" width="0" layer="19" extent="1-1"/>
+<wire x1="-5.08" y1="-3.81" x2="18.62" y2="-1948.19" width="0" layer="19" extent="1-1"/>
 </signal>
 <signal name="!GFIRE">
@@
 <contactref element="IC36" pad="14"/>
 <contactref element="IC37" pad="14"/>
+<contactref element="IC38" pad="14"/>
 <wire x1="3.38" y1="-1788.19" x2="3.38" y2="-1525.19" width="0" layer="19" extent="1-1"/>
 <wire x1="3.38" y1="-1809.19" x2="3.38" y2="-1788.19" width="0" layer="19" extent="1-1"/>
@@
 <contactref element="IC17" pad="2"/>
 <contactref element="V4" pad="6"/>
-<contactref element="IC29" pad="2"/>
-<contactref element="IC29" pad="4"/>
+<contactref element="IC38" pad="5"/>
 <wire x1="9.92" y1="149.19" x2="12.46" y2="149.19" width="0" layer="19" extent="1-1"/>
 <wire x1="12.46" y1="128.19" x2="12.46" y2="149.19" width="0" layer="19" extent="1-1"/>
 <wire x1="9.92" y1="128.19" x2="12.46" y2="128.19" width="0" layer="19" extent="1-1"/>
+<wire x1="2.54" y1="-3.81" x2="9.92" y2="128.19" width="0" layer="19" extent="1-1"/>
 <wire x1="9.92" y1="-1155.81" x2="12.46" y2="149.19" width="0" layer="19" extent="1-1"/>
 <wire x1="20.08" y1="-1119.81" x2="9.92" y2="-1155.81" width="0" layer="19" extent="1-1"/>
-<wire x1="5.73" y1="-1866.81" x2="9.92" y2="-1155.81" width="0" layer="19" extent="1-1"/>
-<wire x1="10.81" y1="-1866.81" x2="5.73" y2="-1866.81" width="0" layer="19" extent="1-1"/>
 </signal>
 <signal name="N$33">
@@
 <wire x1="5.73" y1="-1325.19" x2="8.27" y2="-1325.19" width="0" layer="19" extent="1-1"/>
 </signal>
-<signal name="N$55">
+<signal name="GAMEACTIVE">
 <contactref element="IC22" pad="3"/>
 <contactref element="IC21" pad="13"/>
+<contactref element="IC38" pad="4"/>
 <wire x1="8.27" y1="-1332.81" x2="5.92" y2="-1261.19" width="0" layer="19" extent="1-1"/>
+<wire x1="0" y1="-3.81" x2="5.92" y2="-1261.19" width="0" layer="19" extent="1-1"/>
 </signal>
 <signal name="N$56">
@@
 <wire x1="5.73" y1="-1546.19" x2="8.27" y2="-1546.19" width="0" layer="19" extent="1-1"/>
 </signal>
-<signal name="N$66">
+<signal name="BDEAD">
 <contactref element="IC25" pad="3"/>
 <contactref element="IC26" pad="4"/>
 <contactref element="IC24" pad="4"/>
+<contactref element="IC38" pad="1"/>
 <wire x1="8.27" y1="-1553.81" x2="11" y2="-1532.81" width="0" layer="19" extent="1-1"/>
 <wire x1="10.81" y1="-1619.81" x2="8.27" y2="-1553.81" width="0" layer="19" extent="1-1"/>
+<wire x1="-7.62" y1="-3.81" x2="11" y2="-1532.81" width="0" layer="19" extent="1-1"/>
 </signal>
 <signal name="N$67">
@@
 <wire x1="3.38" y1="-1816.81" x2="3.73" y2="-1831" width="0" layer="19" extent="1-1"/>
 </signal>
-<signal name="N$52">
-<contactref element="IC24" pad="13"/>
-<contactref element="IC27" pad="6"/>
-<wire x1="16.08" y1="-1795.81" x2="5.92" y2="-1525.19" width="0" layer="19" extent="1-1"/>
-</signal>
 <signal name="!GH">
 <contactref element="IC24" pad="12"/>
@@
 <wire x1="8.27" y1="-1859.19" x2="5.73" y2="-1859.19" width="0" layer="19" extent="1-1"/>
 </signal>
-<signal name="N$79">
-<contactref element="C29" pad="2"/>
-</signal>
-<signal name="N$80">
-<contactref element="R40" pad="1"/>
-<contactref element="MOV_POT" pad="1"/>
-<wire x1="2.92" y1="-1909" x2="8" y2="-1927" width="0" layer="19" extent="1-1"/>
-</signal>
 <signal name="N$75">
 <contactref element="IC29" pad="3"/>
@@
 <wire x1="2.54" y1="3.81" x2="11" y2="-1809.19" width="0" layer="19" extent="1-1"/>
 </signal>
+<signal name="!GDEAD">
+<contactref element="IC10" pad="2"/>
+<contactref element="R20" pad="1"/>
+<contactref element="IC22" pad="4"/>
+<contactref element="IC37" pad="8"/>
+<wire x1="31.75" y1="-673.1" x2="31.75" y2="-717.55" width="0" layer="19" extent="1-1"/>
+<wire x1="10.81" y1="-1332.81" x2="31.75" y2="-717.55" width="0" layer="19" extent="1-1"/>
+<wire x1="7.62" y1="3.81" x2="31.75" y2="-673.1" width="0" layer="19" extent="1-1"/>
+</signal>
+<signal name="N$66">
+<contactref element="IC38" pad="3"/>
+<contactref element="IC37" pad="9"/>
+<wire x1="-2.54" y1="-3.81" x2="5.08" y2="3.81" width="0" layer="19" extent="1-1"/>
+</signal>
+<signal name="N$52">
+<contactref element="IC27" pad="6"/>
+<contactref element="IC24" pad="13"/>
+<wire x1="16.08" y1="-1795.81" x2="5.92" y2="-1525.19" width="0" layer="19" extent="1-1"/>
+</signal>
+<signal name="N$80">
+<contactref element="R40" pad="1"/>
+<contactref element="MOV_POT" pad="1"/>
+<wire x1="2.92" y1="-1909" x2="8" y2="-1927" width="0" layer="19" extent="1-1"/>
+</signal>
+<signal name="N$101">
+<contactref element="IC38" pad="6"/>
+<contactref element="IC37" pad="11"/>
+<wire x1="0" y1="3.81" x2="5.08" y2="-3.81" width="0" layer="19" extent="1-1"/>
+</signal>
+<signal name="N$102">
+<contactref element="IC37" pad="10"/>
+<contactref element="IC29" pad="2"/>
+<contactref element="IC29" pad="4"/>
+<wire x1="10.81" y1="-1866.81" x2="5.73" y2="-1866.81" width="0" layer="19" extent="1-1"/>
+<wire x1="2.54" y1="3.81" x2="5.73" y2="-1866.81" width="0" layer="19" extent="1-1"/>
+</signal>
 </signals>

Commit message: -modified the good guy death circuit so it works. I'm not happy with how it works but it works so fuck it -fixed the bad guy death circuit so he can't kill the good guy while he flashes
Parts:
- added IC39: 7404N, 74xx-us:DIL14
- added T7: (no value), transistor:TO92
- moved T1 1674.2 mm to (-1.27, -2010.7)
- moved T2 1671.6 mm to (-1.27, -2023.4)
- moved T3 1669.1 mm to (-1.27, -2036.1)
- moved T4 1666.6 mm to (-1.27, -2048.8)
- moved T5 1664.0 mm to (-1.27, -2061.5)
- moved T6 1661.5 mm to (-1.27, -2074.2)
Connections:
- net N$102 renamed !VRST
- removed net N$101: IC37.11, IC38.6
- new net !BDEAD: IC37.12, IC38.1
- new net N$55: IC38.2, IC39.2
- new net N$79: IC29.1, T7.3
- net !GHIT: now also IC39.1; no longer IC38.2
- net +5V: now also MOV_POT.2; no longer MOV_POT.3
- net BDEAD: now also IC37.13; no longer IC38.1
- net GAMEACTIVE: now also T7.2; no longer IC38.4
- net GND: now also IC39.7, T7.1; no longer IC29.1
- net VCC: now also IC39.14
- net VRST: now also IC37.11; no longer IC38.5

Commit message: -created a scorekeeping circuit
Parts:
- added DIS1, DIS2: HD-F103, display-hp:HDSP-E
- added IC40, IC41: 7490N, 74xx-us:DIL14
- added IC42, IC43: 4511N, 45xx:DIL16
- added R46, R47, R48, R49: 10k, resistor:0207/10
Connections:
- new net N$101: IC40.12, IC40.14, IC42.7
- new net N$102: IC40.9, IC42.1
- new net N$103: IC40.8, IC42.2
- new net N$105: IC41.12, IC41.14, IC43.7
- new net N$106: IC41.9, IC43.1
- new net N$107: IC41.8, IC43.2
- new net N$108: IC41.11, IC43.6
- new net N$109: IC40.11, IC41.1, IC42.6, R47.1
- new net N$110: DIS1.10, IC42.13
- new net N$111: DIS1.9, IC42.12
- new net N$112: DIS1.8, IC42.11
- new net N$113: DIS1.5, IC42.10
- new net N$114: DIS1.4, IC42.9
- new net N$115: DIS1.2, IC42.15
- new net N$116: DIS1.3, IC42.14
- new net N$117: DIS2.10, IC43.13
- new net N$118: DIS2.9, IC43.12
- new net N$119: DIS2.8, IC43.11
- new net N$120: DIS2.5, IC43.10
- new net N$121: DIS2.4, IC43.9
- new net N$122: DIS2.2, IC43.15
- new net N$123: DIS2.3, IC43.14
- new net VDD: IC42.16, IC43.16
- new net VSS: IC42.8, IC43.8
- net +5V: now also IC42.3, IC42.4, IC43.3, IC43.4
- net GND: now also DIS1.1, DIS1.6, DIS1.7, DIS2.1, DIS2.6, DIS2.7, IC40.10, IC40.6, IC40.7, IC41.10, IC41.6, IC41.7, IC42.5, IC43.5, R46.2, R47.2, R48.1, R49.1
- net LOAD: now also IC40.1, R46.1
- net START_PULSE: now also IC40.2, IC40.3, IC41.2, IC41.3, R48.2, R49.2
- net VCC: now also IC40.5, IC41.5

Commit message: -added timing circuit -added scorekeeping circuit
Parts:
- removed T7: (no value), transistor:TO92
- added C36, C37: 10nF, resistor:C025-040X050
- added DIS3, DIS4: HD-F103, display-hp:HDSP-E
- added IC44: 74LS92N, 74xx-us:DIL14
- added IC45, IC46, IC47: 7490N, 74xx-us:DIL14
- added IC48, IC49: 4511N, 45xx:DIL16
- added IC50: 7400N, 74xx-us:DIL14
- added R50, R51, R52, R53: 10k, resistor:0207/10
- added R54, R55: 470, resistor:0207/10
- R30: value 1.5M -> 2.73M
Connections:
- new net !STOP: IC38.10, IC39.8, IC50.4
- new net 1HZ: IC45.11, IC46.1, R50.1
- new net N$104: IC46.12, IC46.14, IC48.7
- new net N$124: IC45.1, IC45.12
- new net N$125: IC46.9, IC48.1
- new net N$126: IC46.8, IC48.2
- new net N$127: IC50.3, IC50.5
- new net N$129: IC47.8, IC49.2
- new net N$130: IC47.11, IC49.6
- new net N$131: IC46.11, IC47.1, IC48.6, R51.1
- new net N$132: DIS3.10, IC48.13
- new net N$133: DIS3.9, IC48.12
- new net N$134: DIS3.8, IC48.11
- new net N$135: DIS3.5, IC48.10
- new net N$136: DIS3.4, IC48.9
- new net N$137: DIS3.2, IC48.15
- new net N$138: DIS3.3, IC48.14
- new net N$139: DIS4.10, IC49.13
- new net N$140: DIS4.9, IC49.12
- new net N$141: DIS4.8, IC49.11
- new net N$142: DIS4.5, IC49.10
- new net N$143: DIS4.4, IC49.9
- new net N$144: DIS4.2, IC49.15
- new net N$145: DIS4.3, IC49.14
- new net N$146: IC38.6, IC38.9
- new net N$147: C37.1, IC50.6
- new net N$148: IC38.12, IC39.4, IC39.5
- new net N$149: C36.1, IC38.11
- new net N$150: C36.2, IC39.3, R54.2
- new net N$151: C37.2, IC39.9, R55.2
- new net RESET_CLOCK: IC39.6, IC46.2, IC46.3, IC47.2, IC47.3, R52.2, R53.2
- new net STA: IC47.12, IC47.14, IC49.7, IC50.1
- new net START_TIMER: IC38.13, IC38.5, IC38.8, IC44.6, IC44.7, IC45.2, IC45.3
- new net STB: IC47.9, IC49.1, IC50.2
- net !START: now also IC38.4
- net !VRST: no longer IC29.4
- net +5V: now also IC48.3, IC48.4, IC49.3, IC49.4
- net GAMEACTIVE: now also IC29.4; no longer T7.2
- net GND: now also DIS3.1, DIS3.6, DIS3.7, DIS4.1, DIS4.6, DIS4.7, IC29.1, IC44.10, IC44.14, IC45.10, IC45.6, IC46.10, IC46.6, IC46.7, IC47.10, IC47.6, IC47.7, IC48.5, IC49.5, IC50.7, R50.2, R51.2, R52.1, R53.1, R54.1, R55.1; no longer T7.1
- net N$79: now also IC44.8, IC45.14; no longer IC29.1, T7.3
- net VCC: now also IC44.5, IC45.5, IC46.5, IC47.5, IC50.14
- net VDD: now also IC48.16, IC49.16
- net VRST: now also IC44.1
- net VSS: now also IC48.8, IC49.8
