File: ambush.brd (EAGLE design)
At the start: 100 x 100 mm, 159 parts, among them IC1 LM555N, IC10 LM555N, IC11 7430N, IC12 7400N, IC13 LM386N-3, IC14 74LS93N, IC15 74LS93N, IC16 7410N, IC17 7402N, IC18 7402N, IC19 7486N, IC2 7404N, IC20 74125N, IC21 7400N, IC22 LM555N, IC23 LM555N, IC24 7400N, IC25 LM555N, IC26 LM555N, IC27 74S20N, IC28 7404N, IC29 LM555N, IC3 LM555N, IC30 7400N, IC31 7475N, IC32 7485N, IC33 7485N, IC34 LM555N, IC35 LM555N, IC36 7402N, IC37 7404N, IC38 7400N, IC39 7404N, IC4 LM555N, IC40 7490N, IC41 7490N, IC42 4511N, IC43 4511N, IC44 74LS92N, IC45 7490N, IC46 7490N, IC47 7490N, IC48 4511N, IC49 4511N, IC5 7404N, IC50 7400N, IC6 74LS93N, IC7 LM555N, IC8 LM555N, IC9 74LS93N, T1 2N3904, T2 2N3904, T3 2N3904, T4 2N3904, T5 2N3904, T6 2N3904, Y1 14.3 MHz

Commit message: -optimized the sound circuitry
Parts:
- removed C1, C10, C11, C14, C15, C2, C3, C7, C8, C9: 100nF, resistor:C025-040X050
- removed IC1, IC10, IC3, IC7, IC8: LM555N, linear:DIL08
- removed R1, R12, R14, R16, R20: 470, resistor:0207/10
- removed R11, R13, R15, R19, R2: 1M, resistor:0207/10
- added C38, C39: 100nF, resistor:C025-040X050
- added IC51: 74116N, 74xx-us:DIL24-6
- added IC52: LM555N, linear:DIL08
- added IC53: 7430N, 74xx-us:DIL14
- added IC54: 7404N, 74xx-us:DIL14
- added R56: 1M, resistor:0207/10
- added R57: 470, resistor:0207/10
- added R58: 10k, resistor:0207/10
- moved T6 2074.2 mm to (-1.27, 0.00)
- moved T5 2061.5 mm to (-1.27, 0.00)
- moved T4 2048.8 mm to (-1.27, 0.00)
- moved T3 2036.1 mm to (-1.27, 0.00)
- moved T2 2023.4 mm to (-1.27, 0.00)
- moved T1 2010.7 mm to (-1.27, 0.00)
Connections:
- removed net !BGFLASH: IC5.4, IC7.2, R14.1
- removed net BGFLASH: IC5.3
- removed net N$1: C1.1, IC3.6, IC3.7, R11.1
- removed net N$2: C7.2, IC3.5
- removed net N$20: C14.1, IC10.6, IC10.7, R19.1
- removed net N$22: C15.2, IC10.5
- removed net N$3: C8.1, IC7.6, IC7.7, R13.1
- removed net N$4: C9.2, IC7.5
- removed net N$5: C2.1, IC1.6, IC1.7, R2.1
- removed net N$6: C10.1, IC8.6, IC8.7, R15.1
- removed net N$7: C3.2, IC1.5
- removed net N$8: C11.2, IC8.5
- new net !BG_FLASH: IC39.12, IC51.8, IC53.12
- new net !SOUND_EN: IC39.10, IC51.14, IC51.15, IC51.2, IC51.3
- new net N$128: C39.1, IC52.6, IC52.7, R56.1
- new net N$152: C38.2, IC52.5
- new net PLAY_SOUND: IC51.1, IC51.13, IC52.3, R58.2
- new net SOUND_EN: IC39.11, IC52.2, IC53.8, R57.1
- net !GDEAD: now also IC51.16, IC53.4; no longer IC10.2, R20.1
- net !GFIRE: now also IC51.6, IC53.6; no longer IC3.2, R12.1
- net !LOAD: now also IC51.10, IC53.11, IC54.2; no longer IC5.2, IC8.2, R16.1
- net !START: now also IC51.4, IC53.5; no longer IC1.2, R1.1
- net +5V: now also IC52.4, IC52.8, IC53.1, IC53.2, IC53.3, R56.2, R57.2; no longer IC1.4, IC1.8, IC10.4, IC10.8, IC3.4, IC3.8, IC7.4, IC7.8, IC8.4, IC8.8, R1.2, R11.2, R12.2, R13.2, R14.2, R15.2, R16.2, R19.2, R2.2, R20.2
- net BG_FLASH: now also IC39.13
- net GND: now also C38.1, C39.2, IC51.12, IC51.18, IC51.20, IC51.22, IC52.1, IC53.7, IC54.7, R58.1; no longer C1.2, C10.2, C11.1, C14.2, C15.1, C2.2, C3.1, C7.1, C8.2, C9.1, IC1.1, IC10.1, IC3.1, IC7.1, IC8.1
- net LOAD: now also IC54.1; no longer IC5.1
- net NOTE1: now also IC51.5; no longer IC1.3
- net NOTE2: now also IC51.7; no longer IC3.3
- net NOTE3: now also IC51.9; no longer IC7.3
- net NOTE4: now also IC51.11; no longer IC8.3
- net NOTE5: now also IC51.17
- net NOTE6: no longer IC10.3
- net VCC: now also IC51.24, IC53.14, IC54.14
