File: ambush.sch (EAGLE design)
At the start: 96 parts, among them IC1 LM555N, IC10 LM555N, IC11 7430N, IC12 7400N, IC13 LM386N-3, IC14 74LS93N, IC15 74LS93N, IC16 7410N, IC17 7402N, IC18 7402N, IC19 7486N, IC2 7404N, IC20 74125N, IC21 7400N, IC22 LM555N, IC23 LM555N, IC24 7400N, IC25 LM555N, IC26 LM555N, IC3 LM555N, IC4 LM555N, IC5 7404N, IC6 74LS93N, IC7 LM555N, IC8 LM555N, IC9 74LS93N, T1 2N3904, T2 2N3904, T3 2N3904, T4 2N3904, T5 2N3904, T6 2N3904, Y1 14.3 MHz

Commit message: -finished control board
Parts:
- added C24, C27, C28, C30: 10nF, resistor:C-US025-040X050
- added C25, C26, C31, C32, C34, C35: 100nF, resistor:C-US025-040X050
- added C29: 47nF, resistor:C-US025-040X050
- added C33: 200nF, resistor:C-US025-040X050
- added IC27: 74S20N, 74xx-us:74S20N
- added IC28, IC37: 7404N, 74xx-us:7404N
- added IC29, IC34, IC35: LM555N, linear:LM555N
- added IC30: 7400N, 74xx-us:7400N
- added IC31: 7475N, 74xx-us:7475N
- added IC32, IC33: 7485N, 74xx-us:7485N
- added IC36: 7402N, 74xx-us:7402N
- added MOV_POT: 500k, pot:3RP/1610N
- added R36: 470k, resistor:R-US_0207/10
- added R37, R42, R43: 1M, resistor:R-US_0207/10
- added R38, R39, R41, R44, R45: 470, resistor:R-US_0207/10
- added R40: 3.3k, resistor:R-US_0207/10
Connections:
- new net !128H: IC27A.I1
- new net !256H: IC27A.I0
- new net !32H: IC27A.I3
- new net !64H: IC27A.I2
- new net !GH: IC24D.I0, IC28A.O
- new net !GV: IC28B.O, IC28C.I, IC30A.I0
- new net BG_FLASH: IC26.Q, IC36B.I0
- new net LOAD\: IC24C.O
- new net N$67: C24.1, IC26.CV
- new net N$68: C25.1, IC26.THR, IC26.TR, R36.2
- new net N$69: IC26.DIS, R36.1, R37.2
- new net N$70: C26.1, IC24B.O
- new net N$71: C26.2, IC2F.I, R38.1
- new net N$72: C27.2, IC24D.O
- new net N$73: IC24B.I1, IC24C.I0, IC2F.O
- new net N$74: C27.1, IC28A.I, R39.1
- new net N$75: IC29.Q, IC30A.I1
- new net N$76: C28.1, IC29.CV
- new net N$77: C30.2, IC30A.O
- new net N$78: C29.1, IC29.DIS, IC29.THR, R40.2
- new net N$79: C29.2
- new net N$80: MOV_POT.A, R40.1
- new net N$81: C30.1, IC28B.I, R41.1
- new net N$82: IC31A.!Q1, IC32A.A0
- new net N$83: IC31A.Q2, IC33A.A0
- new net N$84: IC31A.Q3, IC32A.A2, IC33A.A1
- new net N$85: IC28C.O, IC30B.I1
- new net N$86: IC30B.I0, IC30D.I0, IC32A.A=B_O
- new net N$87: IC28D.I, IC30B.O, IC34.TR
- new net N$88: IC31A.Q4, IC32A.A3, IC33A.A2
- new net N$89: C31.2, IC34.CV
- new net N$90: C32.2, IC35.CV
- new net N$91: C33.2, IC34.DIS, IC34.THR, R42.1
- new net N$92: C34.2, IC35.DIS, IC35.THR, R43.1
- new net N$93: C35.2, IC34.Q, R44.2
- new net N$94: C35.1, IC35.TR, R45.2
- new net N$95: IC30D.I1, IC33A.A=B_O
- new net N$96: IC30C.I1, IC35.Q
- new net N$97: IC30D.O, IC36B.I1
- new net START_PULSE: IC21C.I0, IC22.TR, IC24C.I1, IC2D.O
- net !GHIT: now also IC30C.O
- net +5V: now also IC29.V+, IC34.R, IC34.V+, IC35.R, IC35.V+, MOV_POT.E, R37.1, R42.2, R43.2, R44.1, R45.1
- net 128H: now also IC33A.B3
- net 128V: now also IC32A.B3
- net 16H: now also IC33A.B0
- net 16V: now also IC32A.B0
- net 1V: now also IC31A.D1
- net 2V: now also IC31A.D2
- net 32H: now also IC33A.B1
- net 32V: now also IC32A.B1
- net 4V: now also IC31A.D3
- net 64H: now also IC33A.B2
- net 64V: now also IC32A.B2
- net 8V: now also IC31A.D4
- net GND: now also C24.2, C25.2, C28.2, C31.1, C32.1, C33.1, C34.1, IC29.GND, IC32A.A<B_I, IC32A.A>B_I, IC33A.A3, IC33A.A<B_I, IC33A.A>B_I, IC34.GND, IC35.GND, R38.2, R39.2, R41.2
- net GV=BV: now also IC28D.O, IC30C.I0
- net LOAD: now also IC31A.C12, IC31A.C34
- net N$52: now also IC24D.I1, IC27A.O; no longer IC21C.I0, IC22.TR, IC2D.O
- net N$66: now also IC24B.I0
- net VRST: now also IC29.R, IC29.TR
Other:
- note added: "Control Board"
- moved on the sheet: C19, C20, C21, IC23, R32, R33, R34

Commit message: -finished copying my modified schematics from paper to eagle
Connections:
- new net N$100: IC28E.I, IC36C.O
- new net N$98: IC36B.O, IC36C.I0
- new net N$99: IC36A.O, IC36C.I1
- net !128H: now also IC37A.O
- net !256H: now also IC28F.O
- net !32H: now also IC37C.O
- net !64H: now also IC37B.O
- net !GH: now also IC36A.I0
- net !GV: now also IC36A.I1
- net 128H: now also IC37A.I
- net 256H: now also IC28F.I
- net 32H: now also IC37C.I
- net 64H: now also IC37B.I
- net GAME_VID: now also IC28E.O
Other:
- note added: "Figure Board"
- note added: "Note: I bridged !256H and !128H on my prototype to fix some masking issues on the player's bar. Not sure why it worked, so I'm not including it in the schematic."
- note added: "Sound Board"
- note removed: "Sound Generator"
- moved on the sheet: C31, C32, C33, C34, C35, IC28C, IC28D, IC28E, IC28F, IC30B, IC30C, IC30D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

Commit message: -forgot to credit Heiserman
Other:
- note added: "Ambush TTL Based on schematics by David L. Heiserman from his book How to Design and Build Your Own Custom TV Games Modifications, corrections, and digitization performed by Grant Haack"
Changed lines of the file:
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@@
 <text x="528.32" y="-38.1" size="1.778" layer="94">Horizontal Source Board</text>
 <wire x1="642.62" y1="-40.64" x2="642.62" y2="-109.22" width="0.1524" layer="94" style="shortdash"/>
-<wire x1="642.62" y1="-109.22" x2="449.58" y2="-109.22" width="0.1524" layer="94" style="shortdash"/>
+<wire x1="642.62" y1="-109.22" x2="528.32" y2="-109.22" width="0.1524" layer="94" style="shortdash"/>
 <text x="617.22" y="-104.14" size="1.778" layer="94">Vertical Source Board</text>
+<wire x1="528.32" y1="-109.22" x2="449.58" y2="-109.22" width="0.1524" layer="94" style="shortdash"/>
 <wire x1="449.58" y1="-109.22" x2="342.9" y2="-109.22" width="0.1524" layer="94" style="shortdash"/>
 <wire x1="767.08" y1="71.12" x2="767.08" y2="-109.22" width="0.1524" layer="94" style="shortdash"/>
@@
 <wire x1="177.8" y1="-109.22" x2="177.8" y2="-218.44" width="0.1524" layer="94" style="shortdash"/>
 <wire x1="177.8" y1="-218.44" x2="449.58" y2="-218.44" width="0.1524" layer="94" style="shortdash"/>
-<wire x1="449.58" y1="-218.44" x2="449.58" y2="-109.22" width="0.1524" layer="94" style="shortdash"/>
+<wire x1="449.58" y1="-218.44" x2="449.58" y2="-127" width="0.1524" layer="94" style="shortdash"/>
 <text x="180.34" y="-215.9" size="1.778" layer="94">Figure Board</text>
+<text x="452.12" y="-124.46" size="1.778" layer="94">Ambush TTL
+Based on schematics by David L. Heiserman
+from his book
+How to Design and Build Your Own Custom TV Games
+Modifications, corrections, and digitization performed by Grant Haack</text>
+<wire x1="449.58" y1="-127" x2="449.58" y2="-109.22" width="0.1524" layer="94" style="shortdash"/>
+<wire x1="449.58" y1="-127" x2="528.32" y2="-127" width="0.1524" layer="94" style="shortdash"/>
+<wire x1="528.32" y1="-127" x2="528.32" y2="-109.22" width="0.1524" layer="94" style="shortdash"/>
 </plain>
 <instances>

Commit message: -added a feature so the paddle disappears when the game isn't started -made it so the player can't be killed by the bad guy while the bad guy is flashing
Parts:
- added IC38: 7400N, 74xx-us:7400N
Connections:
- removed net N$55: IC21D.I1, IC22.Q
- removed net N$79: C29.2
- new net !GDEAD: IC10.TR, IC22.R, IC37D.O, R20.1
- new net BDEAD: IC24B.I0, IC25.Q, IC26.R, IC38A.I0
- new net GAMEACTIVE: IC21D.I1, IC22.Q, IC38B.I0
- new net N$101: IC37E.I, IC38B.O
- new net N$102: IC29.R, IC29.TR, IC37E.O
- net !GHIT: now also IC38A.I1; no longer IC10.TR, IC22.R, R20.1
- net GND: now also C29.2
- net N$66: now also IC37D.I, IC38A.O; no longer IC24B.I0, IC25.Q, IC26.R
- net VRST: now also IC38B.I1; no longer IC29.R, IC29.TR
Other:
- moved on the sheet: C27, C28, C29, C30, IC24A, IC24D, IC27A, IC28A, IC28B, IC29, IC30A, MOV_POT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

Commit message: -modified the good guy death circuit so it works. I'm not happy with how it works but it works so fuck it -fixed the bad guy death circuit so he can't kill the good guy while he flashes
Parts:
- added IC39: 7404N, 74xx-us:7404N
- added T7: (no value), transistor:-NPN-TO92
Connections:
- net N$102 renamed !VRST
- removed net N$101: IC37E.I, IC38B.O
- new net !BDEAD: IC37F.O, IC38A.I0
- new net N$55: IC38A.I1, IC39A.O
- new net N$79: IC29.GND, T7.C
- net !GHIT: now also IC39A.I; no longer IC38A.I1
- net +5V: now also MOV_POT.S; no longer MOV_POT.E
- net BDEAD: now also IC37F.I; no longer IC38A.I0
- net GAMEACTIVE: now also T7.B; no longer IC38B.I0
- net GND: now also T7.E; no longer IC29.GND
- net VRST: now also IC37E.I; no longer IC38B.I1
Other:
- moved on the sheet: C28, C29, IC29, IC37D, IC37E, IC38A, R40

Commit message: -created a scorekeeping circuit
Parts:
- added DIS1, DIS2: HD-F103, display-hp:HD-F103
- added IC40, IC41: 7490N, 74xx-us:7490N
- added IC42, IC43: 4511N, 45xx:4511N
- added R46, R47, R48, R49: 10k, resistor:R-US_0207/10
Connections:
- new net N$101: IC40A.CKA, IC40A.QA, IC42A.IA
- new net N$102: IC40A.QB, IC42A.IB
- new net N$103: IC40A.QC, IC42A.IC
- new net N$105: IC41A.CKA, IC41A.QA, IC43A.IA
- new net N$106: IC41A.QB, IC43A.IB
- new net N$107: IC41A.QC, IC43A.IC
- new net N$108: IC41A.QD, IC43A.ID
- new net N$109: IC40A.QD, IC41A.CKB, IC42A.ID, R47.1
- new net N$110: DIS1.A, IC42A.A
- new net N$111: DIS1.B, IC42A.B
- new net N$112: DIS1.C, IC42A.C
- new net N$113: DIS1.D, IC42A.D
- new net N$114: DIS1.E, IC42A.E
- new net N$115: DIS1.F, IC42A.F
- new net N$116: DIS1.G, IC42A.G
- new net N$117: DIS2.A, IC43A.A
- new net N$118: DIS2.B, IC43A.B
- new net N$119: DIS2.C, IC43A.C
- new net N$120: DIS2.D, IC43A.D
- new net N$121: DIS2.E, IC43A.E
- new net N$122: DIS2.F, IC43A.F
- new net N$123: DIS2.G, IC43A.G
- net +5V: now also IC42A.BI, IC42A.LT, IC43A.BI, IC43A.LT
- net GND: now also DIS1.CC, DIS1.CC@1, DIS1.DP, DIS2.CC, DIS2.CC@1, DIS2.DP, IC40A.R9(1), IC40A.R9(2), IC41A.R9(1), IC41A.R9(2), IC42A.LE, IC43A.LE, R46.2, R47.2, R48.1, R49.1
- net LOAD: now also IC40A.CKB, R46.1
- net START_PULSE: now also IC40A.R0(1), IC40A.R0(2), IC41A.R0(1), IC41A.R0(2), R48.2, R49.2
Other:
- note added: "1's Digit"
- note added: "10's Digit"

Commit message: -added timing circuit -added scorekeeping circuit
Parts:
- removed T7: (no value), transistor:-NPN-TO92
- added C36, C37: 10nF, resistor:C-US025-040X050
- added DIS3, DIS4: HD-F103, display-hp:HD-F103
- added IC44: 74LS92N, 74xx-us:74LS92N
- added IC45, IC46, IC47: 7490N, 74xx-us:7490N
- added IC48, IC49: 4511N, 45xx:4511N
- added IC50: 7400N, 74xx-us:7400N
- added R50, R51, R52, R53: 10k, resistor:R-US_0207/10
- added R54, R55: 470, resistor:R-US_0207/10
- R30: value 1.5M -> 2.73M
Connections:
- new net !STOP: IC38C.I1, IC39D.O, IC50B.I0
- new net 1HZ: IC45A.QD, IC46A.CKB, R50.1
- new net N$104: IC46A.CKA, IC46A.QA, IC48A.IA
- new net N$124: IC45A.CKB, IC45A.QA
- new net N$125: IC46A.QB, IC48A.IB
- new net N$126: IC46A.QC, IC48A.IC
- new net N$127: IC50A.O, IC50B.I1
- new net N$129: IC47A.QC, IC49A.IC
- new net N$130: IC47A.QD, IC49A.ID
- new net N$131: IC46A.QD, IC47A.CKB, IC48A.ID, R51.1
- new net N$132: DIS3.A, IC48A.A
- new net N$133: DIS3.B, IC48A.B
- new net N$134: DIS3.C, IC48A.C
- new net N$135: DIS3.D, IC48A.D
- new net N$136: DIS3.E, IC48A.E
- new net N$137: DIS3.F, IC48A.F
- new net N$138: DIS3.G, IC48A.G
- new net N$139: DIS4.A, IC49A.A
- new net N$140: DIS4.B, IC49A.B
- new net N$141: DIS4.C, IC49A.C
- new net N$142: DIS4.D, IC49A.D
- new net N$143: DIS4.E, IC49A.E
- new net N$144: DIS4.F, IC49A.F
- new net N$145: DIS4.G, IC49A.G
- new net N$146: IC38B.O, IC38C.I0
- new net N$147: C37.1, IC50B.O
- new net N$148: IC38D.I0, IC39B.O, IC39C.I
- new net N$149: C36.1, IC38D.O
- new net N$150: C36.2, IC39B.I, R54.2
- new net N$151: C37.2, IC39D.I, R55.2
- new net RESET_CLOCK: IC39C.O, IC46A.R0(1), IC46A.R0(2), IC47A.R0(1), IC47A.R0(2), R52.2, R53.2
- new net STA: IC47A.CKA, IC47A.QA, IC49A.IA, IC50A.I0
- new net START_TIMER: IC38B.I1, IC38C.O, IC38D.I1, IC44A.R0(1), IC44A.R0(2), IC45A.R0(1), IC45A.R0(2)
- new net STB: IC47A.QB, IC49A.IB, IC50A.I1
- net !START: now also IC38B.I0
- net !VRST: no longer IC29.R
- net +5V: now also IC48A.BI, IC48A.LT, IC49A.BI, IC49A.LT
- net GAMEACTIVE: now also IC29.R; no longer T7.B
- net GND: now also DIS3.CC, DIS3.CC@1, DIS3.DP, DIS4.CC, DIS4.CC@1, DIS4.DP, IC29.GND, IC44A.CKA, IC45A.R9(1), IC46A.R9(1), IC46A.R9(2), IC47A.R9(1), IC47A.R9(2), IC48A.LE, IC49A.LE, R50.2, R51.2, R52.1, R53.1, R54.1, R55.1; no longer T7.E
- net N$79: now also IC44A.QD, IC45A.CKA; no longer IC29.GND, T7.C
- net VRST: now also IC44A.CKB
Other:
- note added: "Scorekeeping Board"
- note added: "Timer Board"
- note added: "Timer is set to reset after 30 seconds"
- moved on the sheet: DIS1, DIS2, IC40, IC41, IC42, IC43, R46, R47, R48, R49

Commit message: -optimized the sound circuitry
Parts:
- removed C1, C10, C11, C14, C15, C2, C3, C7, C8, C9: 100nF, resistor:C-US025-040X050
- removed IC1, IC10, IC3, IC7, IC8: LM555N, linear:LM555N
- removed R1, R12, R14, R16, R20: 470, resistor:R-US_0207/10
- removed R11, R13, R15, R19, R2: 1M, resistor:R-US_0207/10
- added C38, C39: 100nF, resistor:C-US025-040X050
- added IC51: 74116N, 74xx-us:74116N
- added IC52: LM555N, linear:LM555N
- added IC53: 7430N, 74xx-us:7430N
- added IC54: 7404N, 74xx-us:7404N
- added R56: 1M, resistor:R-US_0207/10
- added R57: 470, resistor:R-US_0207/10
- added R58: 10k, resistor:R-US_0207/10
Connections:
- removed net !BGFLASH: IC5B.O, IC7.TR, R14.1
- removed net BGFLASH: IC5B.I
- removed net N$1: C1.1, IC3.DIS, IC3.THR, R11.1
- removed net N$2: C7.2, IC3.CV
- removed net N$20: C14.1, IC10.DIS, IC10.THR, R19.1
- removed net N$22: C15.2, IC10.CV
- removed net N$3: C8.1, IC7.DIS, IC7.THR, R13.1
- removed net N$4: C9.2, IC7.CV
- removed net N$5: C2.1, IC1.DIS, IC1.THR, R2.1
- removed net N$6: C10.1, IC8.DIS, IC8.THR, R15.1
- removed net N$7: C3.2, IC1.CV
- removed net N$8: C11.2, IC8.CV
- new net !BG_FLASH: IC39F.O, IC51A.D3, IC53A.I7
- new net !SOUND_EN: IC39E.O, IC51A.G1, IC51A.G2, IC51B.G1, IC51B.G2
- new net N$128: C39.1, IC52.DIS, IC52.THR, R56.1
- new net N$152: C38.2, IC52.CV
- new net PLAY_SOUND: IC51A.CLR, IC51B.CLR, IC52.Q, R58.2
- new net SOUND_EN: IC39E.I, IC52.TR, IC53A.O, R57.1
- net !GDEAD: now also IC51B.D1, IC53A.I3; no longer IC10.TR, R20.1
- net !GFIRE: now also IC51A.D2, IC53A.I5; no longer IC3.TR, R12.1
- net !LOAD: now also IC51A.D4, IC53A.I6, IC54A.O; no longer IC5A.O, IC8.TR, R16.1
- net !START: now also IC51A.D1, IC53A.I4; no longer IC1.TR, R1.1
- net +5V: now also IC52.R, IC52.V+, IC53A.I0, IC53A.I1, IC53A.I2, R56.2, R57.2; no longer IC1.R, IC1.V+, IC10.R, IC10.V+, IC3.R, IC3.V+, IC7.R, IC7.V+, IC8.R, IC8.V+, R1.2, R11.2, R12.2, R13.2, R14.2, R15.2, R16.2, R19.2, R2.2, R20.2
- net BG_FLASH: now also IC39F.I
- net GND: now also C38.1, C39.2, IC51B.D2, IC51B.D3, IC51B.D4, IC52.GND, R58.1; no longer C1.2, C10.2, C11.1, C14.2, C15.1, C2.2, C3.1, C7.1, C8.2, C9.1, IC1.GND, IC10.GND, IC3.GND, IC7.GND, IC8.GND
- net LOAD: now also IC54A.I; no longer IC5A.I
- net NOTE1: now also IC51A.Q1; no longer IC1.Q
- net NOTE2: now also IC51A.Q2; no longer IC3.Q
- net NOTE3: now also IC51A.Q3; no longer IC7.Q
- net NOTE4: now also IC51A.Q4; no longer IC8.Q
- net NOTE5: now also IC51B.Q1
- net NOTE6: no longer IC10.Q
Other:
- moved on the sheet: IC5C, IC5D, IC5E, IC5F
